Commit message: use joint_state_pub random

File: src/fun4_description/robot/visual/my-robot.xacro (robot description, xacro)
@@ -44,11 +44,11 @@
         <dynamic damping="0.1" friction="0.05" />
     </joint>
-    <joint name="link_3_end_effector" type="revolute">
+    <joint name="link_3_end_effector" type="fixed">
         <parent link="link_3" />
         <child link="end_effector" />
         <origin xyz="0.280 0 0" rpy="${pi/2} 0 ${pi/2}" />
-        <axis xyz="0 0 1" />
+        <!-- <axis xyz="0 0 1" />
         <limit effort="100" lower="${-pi}" upper="${pi}" velocity="100" />
-        <dynamic damping="0.1" friction="0.05" />
+        <dynamic damping="0.1" friction="0.05" /> -->
     </joint>
 </robot>
