Commit message: finish end_effector_pose

File: install/fun4_description/share/fun4_description/robot/visual/my-robot.xacro (robot description, xacro)
@@ -1,7 +1,84 @@
 <?xml version="1.0"?>
 <robot xmlns:xacro="http://www.ros.org/wiki/xacro" name="example">
-<!-- variable -->
+  <link name="link_0">
+    <visual>
+      <geometry>
+        <mesh filename="package://fun4_description/meshes/link_0.stl"/>
+      </geometry>
+    </visual>
+  </link>
+  <link name="link_1">
+    <visual>
+      <geometry>
+        <mesh filename="package://fun4_description/meshes/link_1.stl"/>
+      </geometry>
+    </visual>
+  </link>
+  <joint name="joint_1" type="revolute">
+    <parent link="link_0"/>
+    <child link="link_1"/>
+    <origin xyz="0 0 0.2" rpy="0 0 0"/>
+    <axis xyz="0 0 1"/>
+    <limit
+      lower="-3.1459"
+      upper="3.1459"
+      velocity="1000.0"
+      effort="1000.0"/>
+  </joint>
+  <link name="link_2">
+    <visual>
+      <origin xyz="0.0 0.0 0.0" rpy="0 0 ${-3.14/2}"/>
+      <geometry>
+        <mesh filename="package://fun4_description/meshes/link_2.stl"/>
+      </geometry>
+    </visual>
+  </link>
+  <joint name="joint_2" type="revolute">
+    <parent link="link_1"/>
+    <child link="link_2"/>
+    <origin xyz="0.0 -0.12 0.0" rpy="${-3.14/2} 0 0"/>
+    <axis xyz="0 0 1"/>
+    <limit
+      lower="-3.1459"
+      upper="3.1459"
+      velocity="1000.0"
+      effort="1000.0"/>
+  </joint>
+  <link name="link_3">
+    <visual>
+      <origin xyz="0.0 0.0 0.0" rpy="0 0 ${-3.14/2}"/>
+      <geometry>
+        <mesh filename="package://fun4_description/meshes/link_3.stl"/>
+      </geometry>
+    </visual>
+  </link>
+  <joint name="joint_3" type="revolute">
+    <parent link="link_2"/>
+    <child link="link_3"/>
+    <origin xyz="0.0 -0.25 0.1" rpy="0 0 0"/>
+    <axis xyz="0 0 1"/>
+    <limit
+      lower="-3.1459"
+      upper="3.1459"
+      velocity="1000.0"
+      effort="1000.0"/>
+  </joint>
+  <link name="end_effector">
+    <visual>
+      <origin xyz="0.0 0.0 0.0" rpy="0 0 0"/>
+      <geometry>
+        <mesh filename="package://fun4_description/meshes/end_effector.stl"/>
+      </geometry>
+    </visual>
+  </link>
+  <joint name="joint_end_effector" type="fixed">
+    <parent link="link_3"/>
+    <child link="end_effector"/>
+    <origin xyz="0.0 -0.28 0.0" rpy="${3.14/2} 0 0"/>
+  </joint>
+</robot>
+<!-- ////////////////////////////////////////////////////////////////////////////////////////////// -->
+<!-- <robot xmlns:xacro="http://www.ros.org/wiki/xacro" name="example">
     <xacro:property name="arm_base_length" value="0.1" />
-<!-- link -->
     <xacro:macro name="arm_link" params="prefix">
         <link name="${prefix}">
@@ -19,36 +96,29 @@
     <xacro:arm_link prefix="link_3"/>
     <xacro:arm_link prefix="end_effector"/>
-<!-- joint -->
-    <joint name="link_0_link_1" type="revolute">
+    <joint name="joint_1" type="revolute">
         <parent link="link_0" />
         <child link="link_1" />
-        <origin xyz="0 0 0.24" rpy="0 0 0" />
+        <origin xyz="0 0 0.2" rpy="0 0 0" />
         <axis xyz="0 0 1" />
-        <limit effort="100" lower="${-pi}" upper="${pi}" velocity="100" />
-        <dynamic damping="0.1" friction="0.05" />
+        <limit effort="1000" lower="${-pi}" upper="${pi}" velocity="1000" />
     </joint>
-    <joint name="link_1_link_2" type="revolute">
+    <joint name="joint_2" type="revolute">
         <parent link="link_1" />
         <child link="link_2" />
         <origin xyz="0 -0.12 0" rpy="${-pi/2} ${-pi/2} 0" />
         <axis xyz="0 0 1" />
-        <limit effort="100" lower="${-pi}" upper="${pi}" velocity="100" />
-        <dynamic damping="0.1" friction="0.05" />
+        <limit effort="1000" lower="${-pi}" upper="${pi}" velocity="1000" />
     </joint>
-    <joint name="link_2_link_3" type="revolute">
+    <joint name="joint_3" type="revolute">
         <parent link="link_2" />
         <child link="link_3" />
         <origin xyz="0.25 0 0.10" rpy="0 0 0" />
         <axis xyz="0 0 1" />
-        <limit effort="100" lower="${-pi}" upper="${pi}" velocity="100" />
-        <dynamic damping="0.1" friction="0.05" />
+        <limit effort="1000" lower="${-pi}" upper="${pi}" velocity="1000" />
     </joint>
-    <joint name="link_3_end_effector" type="fixed">
+    <joint name="joint_end_effector" type="fixed">
         <parent link="link_3" />
         <child link="end_effector" />
         <origin xyz="0.280 0 0" rpy="${pi/2} 0 ${pi/2}" />
-        <!-- <axis xyz="0 0 1" />
-        <limit effort="100" lower="${-pi}" upper="${pi}" velocity="100" />
-        <dynamic damping="0.1" friction="0.05" /> -->
     </joint>
-</robot>
+</robot> -->

Commit message: ik node finish

File: install/fun4_description/share/fun4_description/robot/visual/my-robot.xacro (robot description, xacro)
@@ -1,124 +1,72 @@
 <?xml version="1.0"?>
 <robot xmlns:xacro="http://www.ros.org/wiki/xacro" name="example">
-  <link name="link_0">
-    <visual>
-      <geometry>
-        <mesh filename="package://fun4_description/meshes/link_0.stl"/>
-      </geometry>
-    </visual>
-  </link>
-  <link name="link_1">
-    <visual>
-      <geometry>
-        <mesh filename="package://fun4_description/meshes/link_1.stl"/>
-      </geometry>
-    </visual>
-  </link>
-  <joint name="joint_1" type="revolute">
-    <parent link="link_0"/>
-    <child link="link_1"/>
-    <origin xyz="0 0 0.2" rpy="0 0 0"/>
-    <axis xyz="0 0 1"/>
-    <limit
-      lower="-3.1459"
-      upper="3.1459"
-      velocity="1000.0"
-      effort="1000.0"/>
-  </joint>
-  <link name="link_2">
-    <visual>
-      <origin xyz="0.0 0.0 0.0" rpy="0 0 ${-3.14/2}"/>
-      <geometry>
-        <mesh filename="package://fun4_description/meshes/link_2.stl"/>
-      </geometry>
-    </visual>
-  </link>
-  <joint name="joint_2" type="revolute">
-    <parent link="link_1"/>
-    <child link="link_2"/>
-    <origin xyz="0.0 -0.12 0.0" rpy="${-3.14/2} 0 0"/>
-    <axis xyz="0 0 1"/>
-    <limit
-      lower="-3.1459"
-      upper="3.1459"
-      velocity="1000.0"
-      effort="1000.0"/>
-  </joint>
-  <link name="link_3">
-    <visual>
-      <origin xyz="0.0 0.0 0.0" rpy="0 0 ${-3.14/2}"/>
-      <geometry>
-        <mesh filename="package://fun4_description/meshes/link_3.stl"/>
-      </geometry>
-    </visual>
-  </link>
-  <joint name="joint_3" type="revolute">
-    <parent link="link_2"/>
-    <child link="link_3"/>
-    <origin xyz="0.0 -0.25 0.1" rpy="0 0 0"/>
-    <axis xyz="0 0 1"/>
-    <limit
-      lower="-3.1459"
-      upper="3.1459"
-      velocity="1000.0"
-      effort="1000.0"/>
-  </joint>
-  <link name="end_effector">
-    <visual>
-      <origin xyz="0.0 0.0 0.0" rpy="0 0 0"/>
-      <geometry>
-        <mesh filename="package://fun4_description/meshes/end_effector.stl"/>
-      </geometry>
-    </visual>
-  </link>
-  <joint name="joint_end_effector" type="fixed">
-    <parent link="link_3"/>
-    <child link="end_effector"/>
-    <origin xyz="0.0 -0.28 0.0" rpy="${3.14/2} 0 0"/>
-  </joint>
+    <xacro:property name="pi" value="3.14159265359" />
+    <link name="link_0">
+        <visual>
+            <origin rpy="0 0 0" xyz="0.0 0.0 0.0" />
+            <geometry>
+                <mesh filename="package://fun4_description/meshes/link_0.stl" />
+            </geometry>
+        </visual>
+    </link>
+    <link name="link_1">
+        <visual>
+            <origin rpy="0 0 0" xyz="0.0 0.0 0.0" />
+            <geometry>
+                <mesh filename="package://fun4_description/meshes/link_1.stl" />
+            </geometry>
+        </visual>
+    </link>
+    <joint name="joint_1" type="revolute">
+        <origin xyz="0.0 0.0 0.2" rpy="0.0 0.0 0.0"/>
+        <parent link="link_0"/>
+        <child link="link_1"/>
+        <axis xyz="0.0 0.0 1.0"/>
+        <limit lower="${-pi}" upper="${pi}" effort="100.0" velocity="100.0"/>
+    </joint>
+    <link name="link_2">
+        <visual>
+            <origin rpy="${pi} 0 0" xyz="0.0 0.0 0.0" />
+            <geometry>
+                <mesh filename="package://fun4_description/meshes/link_2.stl" />
+            </geometry>
+        </visual>
+    </link>
+    <joint name="joint_2" type="revolute">
+        <origin xyz="0.0 -0.12 0.0" rpy="1.5708 0 0"/>
+        <parent link="link_1"/>
+        <child link="link_2"/>
+        <axis xyz="0.0 0.0 1.0"/>
+        <limit lower="${-pi}" upper="${pi}" effort="100.0" velocity="100.0"/>
+    </joint>
+    <link name="link_3">
+        <visual>
+            <origin rpy="${pi} 0 0" xyz="0.0 0.0 0.0" />
+            <geometry>
+                <mesh filename="package://fun4_description/meshes/link_3.stl" />
+            </geometry>
+        </visual>
+    </link>
+    <joint name="joint_3" type="revolute">
+        <origin xyz="0.25 0.0 -0.1" rpy="0.0 0.0 0.0"/>
+        <parent link="link_2"/>
+        <child link="link_3"/>
+        <axis xyz="0.0 0.0 1.0"/>
+        <limit lower="${-pi}" upper="${pi}" effort="100.0" velocity="100.0"/>
+    </joint>
+    <link name="end_effector">
+        <visual>
+            <origin rpy="0 1.57 0" xyz="0.0 0.0 0.0" />
+            <geometry>
+                <mesh filename="package://fun4_description/meshes/end_effector.stl" />
+            </geometry>
+        </visual>
+    </link>
+    <joint name="joint_4" type="fixed">
+        <origin xyz="0.28 0.0 0.0" rpy="0.0 0.0 0.0"/>
+        <parent link="link_3"/>
+        <child link="end_effector"/>
+        <axis xyz="0.0 0.0 0.0"/>
+        <limit lower="0.0" upper="${2*pi}" effort="100.0" velocity="100.0"/>
+    </joint>
 </robot>
-<!-- ////////////////////////////////////////////////////////////////////////////////////////////// -->
-<!-- <robot xmlns:xacro="http://www.ros.org/wiki/xacro" name="example">
-    <xacro:property name="arm_base_length" value="0.1" />
-    <xacro:macro name="arm_link" params="prefix">
-        <link name="${prefix}">
-            <visual>
-              <origin rpy="0 0 0" xyz="0 0 0"/>
-              <geometry>
-                <mesh filename="package://example_description/meshes/${prefix}.stl"/>
-              </geometry>
-            </visual>
-          </link>
-    </xacro:macro>
-    <xacro:arm_link prefix="link_0"/>
-    <xacro:arm_link prefix="link_1"/>
-    <xacro:arm_link prefix="link_2"/>
-    <xacro:arm_link prefix="link_3"/>
-    <xacro:arm_link prefix="end_effector"/>
-    <joint name="joint_1" type="revolute">
-        <parent link="link_0" />
-        <child link="link_1" />
-        <origin xyz="0 0 0.2" rpy="0 0 0" />
-        <axis xyz="0 0 1" />
-        <limit effort="1000" lower="${-pi}" upper="${pi}" velocity="1000" />
-    </joint>
-    <joint name="joint_2" type="revolute">
-        <parent link="link_1" />
-        <child link="link_2" />
-        <origin xyz="0 -0.12 0" rpy="${-pi/2} ${-pi/2} 0" />
-        <axis xyz="0 0 1" />
-        <limit effort="1000" lower="${-pi}" upper="${pi}" velocity="1000" />
-    </joint>
-    <joint name="joint_3" type="revolute">
-        <parent link="link_2" />
-        <child link="link_3" />
-        <origin xyz="0.25 0 0.10" rpy="0 0 0" />
-        <axis xyz="0 0 1" />
-        <limit effort="1000" lower="${-pi}" upper="${pi}" velocity="1000" />
-    </joint>
-    <joint name="joint_end_effector" type="fixed">
-        <parent link="link_3" />
-        <child link="end_effector" />
-        <origin xyz="0.280 0 0" rpy="${pi/2} 0 ${pi/2}" />
-    </joint>
-</robot> -->

Commit message: update ipk,teleop
left adjust custom service

File: install/fun4_description/share/fun4_description/robot/visual/my-robot.xacro (robot description, xacro)
@@ -34,5 +34,5 @@
     </link>
     <joint name="joint_2" type="revolute">
-        <origin xyz="0.0 -0.12 0.0" rpy="1.5708 0 0"/>
+        <origin xyz="0.0 -0.12 0.0" rpy="${pi/2} ${-pi/2} 0"/>
         <parent link="link_1"/>
         <child link="link_2"/>
@@ -49,5 +49,5 @@
     </link>
     <joint name="joint_3" type="revolute">
-        <origin xyz="0.25 0.0 -0.1" rpy="0.0 0.0 0.0"/>
+        <origin xyz="0.25 0.0 -0.1" rpy="0.0 0.0 ${pi/2}"/>
         <parent link="link_2"/>
         <child link="link_3"/>
